File: .MAIN_PCB/MAIN_WATERING/MAIN_WATERING.kicad_pcb (KiCad board)
At the start: 2 copper layers, 32.5 x 35.5 mm, 5 parts, among them J1 Conn_01x04_Pin, SW1 SW_Push, U1 XIAO-ESP32-C3-SMD

Commit message: fixed drill holes
Other:
- board size 32.5 x 35.5 mm -> 35.5 x 37 mm
Changed lines of the file:
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@@
 	)
 	(gr_rect
-		(start 155 80)
-		(end 187.5 115.5)
+		(start 153 79.5)
+		(end 188.5 116.5)
 		(stroke
 			(width 0.05)
+			(type default)
+		)
+		(fill no)
+		(layer "Edge.Cuts")
+	)
+	(gr_circle
+		(center 154.5 81)
+		(end 154.5 82)
+		(stroke
+			(width 0.05)
+			(type default)
+		)
+		(fill no)
+		(layer "Edge.Cuts")
+	)
+	(gr_circle
+		(center 154.5 114)
+		(end 154.5 115)
+		(stroke
+			(width 0.05)
+			(type default)
+		)
+		(fill no)
+		(layer "Edge.Cuts")
+	)
+	(gr_circle
+		(center 185.5 81)
+		(end 185.5 82)
+		(stroke
+			(width 0.05)
+			(type default)
+		)
+		(fill no)
+		(layer "Edge.Cuts")
+	)
+	(gr_circle
+		(center 187 114)
+		(end 187 115)
+		(stroke
+			(width 0.05)
